File: hardware/CC1125_Transceiver/CC1125_Transceiver.kicad_pcb (KiCad board)
At the start: 4 copper layers, 67 x 28.8 mm, 79 parts, among them IC1 CC1125RHBT, IC2 GALI-74+, IC3 TLV61046ADBVT, IC4 TLV75801PDRVR, J1 SMA_Ant, J2 Conn_02x03_Counter_Clockwise, J4 USB_C_Receptacle_USB2.0_14P, U2 STM32L412K8Ux, Y1 ECS-TXO-32CSMV-400-BN-TR, Y2 40MHz

Commit message: finalised
Parts:
- added C38: 220n, Capacitor_SMD:C_0402_1005Metric_Pad0.74x0.62mm_HandSolder, F.Cu at (111.0, 88.2)
- added G***: LOGO, LOGO, F.Cu at (137.2, 88.2)
- added TP1: TestPoint_Small, TestPoint:TestPoint_THTPad_D2.0mm_Drill1.0mm, F.Cu at (92.8, 107.8)
- added TP2: TestPoint_Small, TestPoint:TestPoint_THTPad_D2.0mm_Drill1.0mm, F.Cu at (108.0, 106.0)
- J2: footprint Connector_PinHeader_1.00mm:PinHeader_2x03_P1.00mm_Vertical_SMD -> Connector_PinHeader_2.54mm:PinHeader_2x03_P2.54mm_Vertical_SMD
- J4: value USB_C_Receptacle_USB2.0_14P -> USB4216-03-A
- R1, R2: footprint Resistor_SMD:R_0402_1005Metric_Pad0.72x0.64mm_HandSolder -> Resistor_SMD:R_0603_1608Metric_Pad0.98x0.95mm_HandSolder
- moved J2 8.66 mm to (101.0, 104.0), turned to 0 degrees
- moved C17 1.60 mm to (112.0, 88.2)
- moved C24 1.51 mm to (109.0, 88.2), turned to 90 degrees
- moved J1 1.50 mm to (140.1, 99.2)
- moved C31 1.47 mm to (85.0, 104.0)
- moved C15 1.10 mm to (110.0, 88.2)
- moved C10 0.57 mm to (126.1, 104.6)
- moved R2 0.43 mm to (125.0, 103.5)
- moved R1 0.18 mm to (111.2, 103.2)
Connections:
- net /Filt2 renamed /Rx/Tx
- net Net-(IC1-RBIAS) renamed /RBIAS
- IC1 pad 26: +3V3 -> Net-(IC1-DCPL_PFD_CHP)
- J2 pad 2: /CC_Resetn -> /SPI_CSN
- J2 pad 6: /SPI_CSN -> /CC_Resetn
- J4 pad A8: (no net) -> unconnected-(J4-SBU1-PadA8)
- J4 pad B8: (no net) -> unconnected-(J4-SBU2-PadB8)
- R11 pad 1: unconnected-(R11-Pad1) -> /LED_STATUS
- U2 pad 18: unconnected-(U2-PA8-Pad18) -> /LED_STATUS
- U2 pad 6: unconnected-(U2-PA0-Pad6) -> /SPI_CSN
- U2 pad 9: unconnected-(U2-PA3-Pad9) -> /CC_Resetn
Routing:
- net GND: track 18.7 -> 102.9 mm, vias 15 -> 51
- net +7V: track 16.7 -> 80.2 mm
- net +3V3: track 26.8 -> 58.3 mm, vias 7 -> 18
- net /CC_Resetn: track 3.40 -> 31.7 mm, vias 2 -> 3
- net VUSB: track 14.2 -> 41.5 mm
- net /SPI_MISO: track 5.75 -> 30.4 mm, vias 3 -> 2
- net /SPI_SCK: track 4.75 -> 26.5 mm, vias 3 -> 2
- net /SPI_MOSI: track 6.21 -> 27.7 mm, vias 3 -> 2
- net /uc_Reset: track 2.05 -> 18.0 mm, vias 1 -> 2
- net /SPI_CSN: track 6.30 -> 21.4 mm
- net /Anten: track 1.60 -> 15.7 mm
- net Net-(IC1-EXT_XOSC): track 0.00 -> 9.02 mm
- net Net-(IC1-XOSC_Q1): track 0.00 -> 6.95 mm
- net Net-(IC1-XOSC_Q2): track 0.00 -> 5.63 mm
- net /LED_STATUS: track 0.00 -> 5.10 mm
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- added copper zone on F.Cu, net +3V3
- added copper zone on In1.Cu, net +3V3
Other:
- board size 67 x 28.8 mm -> 67.5 x 28.8 mm
- board text added: "3V3"
- board text added: "Entwicklung Resilienter Elektronik-Systeme"
- board text added: "MO CS CK MI GN RS"
- board text added: "PA.V"
- board text added: "V1.0 von Fynn Gewiese"
- board text removed: "V1.0 Gewiese"
