File: hardware/CC1125_Transceiver/CC1125_Transceiver.kicad_sch (KiCad schematic)
At the start: 85 parts, among them IC1 CC1125RHBT, IC2 GALI-74+, IC3 TLV61046ADBVT, IC4 TLV75801PDRVR, J1 SMA_Ant, J2 Conn_02x03_Counter_Clockwise, J4 USB_C_Receptacle_USB2.0_14P, U2 STM32L412K8Ux, Y1 ECS-TXO-32CSMV-400-BN-TR, Y2 40MHz

Commit message: finalised
Parts:
- removed J4: USB_C_Receptacle_USB2.0_14P, libary:USB421603A, symbol Connector:USB_C_Receptacle_USB2.0_14P
- added J4: USB4216-03-A, symbol Connector:USB_C_Receptacle_USB2.0_16P
- added TP1, TP2: TestPoint_Small, TestPoint:TestPoint_THTPad_D2.0mm_Drill1.0mm, symbol Connector:TestPoint_Small
- C10, C2: value C -> 100n
- D1, V1, V2, V3, V4: now not fitted; now left out of the parts list
- D2, D3, D4: value ~ -> (none)
- J2: footprint PinHeader_2x03_P1.00mm_Vertical_SMD -> Connector_PinHeader_2.54mm:PinHeader_2x03_P2.54mm_Vertical_SMD
- L1, L9: value L -> 220n
- R1: value R -> 22; footprint Resistor_SMD:R_0402_1005Metric_Pad0.72x0.64mm_HandSolder -> Resistor_SMD:R_0603_1608Metric_Pad0.98x0.95mm_HandSolder
- R2: footprint Resistor_SMD:R_0402_1005Metric_Pad0.72x0.64mm_HandSolder -> Resistor_SMD:R_0603_1608Metric_Pad0.98x0.95mm_HandSolder
- R8: value 1M -> 100k
- R9: value ToDo -> 20k
Connections:
- net +3V3: now also TP1.1
- net +7V: now also TP2.1
- net CC_Resetn: now also J2.6 (Pin_6), U2.9 (PA3); no longer J2.2 (Pin_2)
- net GND: now also J4.A1 (GND), J4.A12 (GND), J4.B1 (GND), J4.B12 (GND), J4.SH (SHIELD)
- net SPI_CSN: now also J2.2 (Pin_2), U2.6 (PA0); no longer J2.6 (Pin_6)
- net USB_DN: now also J4.A7 (D-), J4.B7 (D-)
- net USB_DP: now also J4.A6 (D+), J4.B6 (D+)
- net at C37.1, R16.1: now also J4.A4 (VBUS), J4.A9 (VBUS), J4.B4 (VBUS), J4.B9 (VBUS)
- net at R6.1: now also J4.A5 (CC1)
- net at R7.1: now also J4.B5 (CC2)
- net LED_STATUS: now reaches U2.18 (PA8)
- net LED_STATUS: now also R11.1
- net RBIAS: now reaches IC1.14 (RBIAS), R3.1
- no-connect marks 0 -> 2
Other:
- moved on the sheet: C22, C23, C24, C25, C26, C38, D2, R11, R3, Y2
